File: hardware/fk-core.sch (KiCad schematic (older format))
At the start: 130 parts, among them J1 RF-SMA-EDGE, J10 S2B-PH-SM4-TB, J11 RF-SMA-EDGE, J12 CONN_01x02, J13 CONN_01x06, J14 CONN_01x02, J2 CONN_01x02, J3 S2B-PH-SM4-TB, J4 Conn_01x01, J5 CONN_01x03_SERIAL, J6 CONN_01x05, J7 CONN_02x05_SWD, J8 CONN_01x02, J9 MICRO-USB, M1 MOUNT_HOLE, M10 FIDUCIAL, M11 FIDUCIAL, M2 FIDUCIAL, M3 MOUNT_HOLE, M4 MOUNT_HOLE, M5 FIDUCIAL, M6 MOUNT_HOLE, M7 MICRO-SD, M8 FIDUCIAL, M9 FIDUCIAL, Q1 2N7002LT1G, SW1 SPNO, SW2 SPNO, U1 ATWINC1500-MR210PA, U10 FGPMMOPA6H, U11 MAX1704XX, U12 TPS2052B, U13 SK6812, U14 MCP1700T-3302E/MB, U2 ATSAMD21G18A-AU, U3 RFM95W, U4 24AA02E64, U5 S25FL116K0XMFI041, U6 BQ24074RGTT, U7 PCF8523, U8 TL5209, U9 TL5209, Y1 FC-135, Y2 FC-135

Commit message: transitioning to a hierarchical schematic
Parts:
- removed BT1: BATTERY_CELL, conservify:BAT_CR1210, symbol fk-core-rescue:BATTERY_CELL-conservify
- removed C11, C13, C15, C16, C18, C32, C33: 100nF, conservify:CAP-0603, symbol fk-core-rescue:CAPACITOR_CERAMIC-conservify
- removed C17, C22, C24, C34, C35: 10uF, conservify:CAP-0603, symbol fk-core-rescue:CAPACITOR_CERAMIC-conservify
- removed C2, C31: 47uF, conservify:CAP-0603, symbol fk-core-rescue:CAPACITOR_CERAMIC-conservify
- removed C26, C27: 1uF, conservify:CAP-0603, symbol fk-core-rescue:CAPACITOR_CERAMIC-conservify
- removed C28: 10nF, conservify:CAP-0603, symbol fk-core-rescue:CAPACITOR_CERAMIC-conservify
- removed C29: 470pF, conservify:CAP-0603, symbol fk-core-rescue:CAPACITOR_CERAMIC-conservify
- removed C30: 2.2uF, conservify:CAP-0603, symbol fk-core-rescue:CAPACITOR_CERAMIC-conservify
- removed D11: Red, conservify:LED-0603, symbol fk-core-rescue:LED_SINGLE-conservify
- removed D2: Green, conservify:LED-0603, symbol fk-core-rescue:LED_SINGLE-conservify
- removed D3: Yellow, conservify:LED-0603, symbol fk-core-rescue:LED_SINGLE-conservify
- removed J1, J11: RF-SMA-EDGE, conservify:RF-SMA-EDGE, symbol fk-core-rescue:RF_SMA_EDGE-conservify
- removed J12, J14, J2: CONN_01x02, conservify:SJ_OPEN, symbol fk-core-rescue:CONN_01x02-conservify
- removed J13: CONN_01x06, conservify:JST_SH_BM06B-SRSS-TB_1x06-1MP_P1.00mm_Vertical, symbol fk-core-rescue:CONN_01x06-conservify
- removed J4: Conn_01x01, conservify:Socket_Strip_Straight_1x01_Pitch2.54mm, symbol fk-core-rescue:CONN_01x01-conservify
- removed J6: CONN_01x05, conservify:Molex_CLIK-Mate_502382-0570_1x05_P1.25mm_Vertical, symbol fk-core-rescue:CONN_01x05-conservify
- removed L3: BLM18KG221SN1D, conservify:IND-0603, symbol fk-core-rescue:INDUCTOR-conservify
- removed M7: MICRO-SD, conservify:MICRO-SD, symbol fk-core-rescue:MICRO_SD-conservify
- removed R1, R13, R18, R19, R2: 100K, conservify:RES-0603, symbol fk-core-rescue:RESISTOR-conservify
- removed R14: 165.7K, conservify:RES-0603, symbol fk-core-rescue:RESISTOR-conservify
- removed R15, R16, R6, R7: 10K, conservify:RES-0603, symbol fk-core-rescue:RESISTOR-conservify
- removed R20: ?, conservify:RES-0603, symbol fk-core-rescue:RESISTOR-conservify
- removed R35, R36, R42, R43: 4.7K, conservify:RES-0603, symbol fk-core-rescue:RESISTOR-conservify
- removed R37, R39, R4, R40, R5: 1K, conservify:RES-0603, symbol fk-core-rescue:RESISTOR-conservify
- removed R41: 180R, conservify:RES-0603, symbol fk-core-rescue:RESISTOR-conservify
- removed U1: ATWINC1500-MR210PA, conservify:ATMEL_ATWINC1500-MR210PA, symbol fk-core-rescue:ATWINC1500_MR210PA-conservify
- removed U10: FGPMMOPA6H, conservify:FGPMMOPA6H, symbol fk-core-rescue:FGPMMOPA6H-conservify
- removed U11: MAX1704XX, conservify:DFN-8-1EP_3x2mm_Pitch0.5mm, symbol fk-core-rescue:MAX1704XX-conservify
- removed U12: TPS2052B, conservify:SOIC-8-N, symbol fk-core-rescue:TPS2052B-conservify
- removed U14: MCP1700T-3302E/MB, conservify:SOT-89, symbol fk-core-rescue:MCP1700T-XXX2E-conservify
- removed U3: RFM95W, conservify:RFM9xW, symbol fk-core-rescue:RFM9xW-conservify
- removed U4: 24AA02E64, conservify:SOT-23-5_HandSoldering, symbol fk-core-rescue:24AA02E64-conservify
- removed U5: S25FL116K0XMFI041, conservify:SOIC-8-N-WIDE, symbol fk-core-rescue:S25FL1xxK0XM-conservify
- removed U7: PCF8523, conservify:SOIC-8-N, symbol fk-core-rescue:PCF8523-conservify
- removed U9: TL5209, conservify:SOIC-8-N, symbol fk-core-rescue:TL5209-conservify
- removed Y2: FC-135, conservify:ABS07, symbol fk-core-rescue:CRYSTAL-conservify
Connections:
- net labels removed: GPS_3V3, GPS_FIX, MODULE_3V3, PERIPH_3V3
- wire segments 561 -> 311
- no-connect marks 41 -> 20
Other:
- note removed: "1. All capacitors are NP0/COG 50V unless specified.\n2. All resistors are 62.5mW 1% unless specified."
- note removed: "16Mbit = 2Mbytes"
- note removed: "24AA02E64 DEVICE ID\n"
- note removed: "BREAKOUT"
- note removed: "GPS"
- note removed: "I2C PULLUP\n"
- note removed: "LED"
- note removed: "LEDS"
- note removed: "LIPO GAUGE"
- note removed: "MCU"
- note removed: "NOTES"
- note removed: "PERIPHERALS"
- note removed: "POWER MANAGEMENT (3V3 REGULATOR)"
- note removed: "RFM95W\n"
- note removed: "RTC"
- note removed: "SD"
- note removed: "SERIAL FLASH"
- note removed: "SWD/JTAG"
- note removed: "WIFI"
